File: LaserNetworkAdaptor/LaserNetworkAdaptor.kicad_pcb (KiCad board)
At the start: 2 copper layers, 19 x 32.6 mm, 5 parts, among them J1 RJ45, J2 Conn_01x10_Male

Commit message: updated text
Other:
- board text removed: "MALWARE SUBSTITUTE"
